File: kicad/solar-light-charlie-boost/solar-light-charlie-boost.kicad_sch (KiCad schematic)
At the start: 32 parts, among them J2 Conn_01x08_Socket, J3 Conn_01x03_Pin, J4 Conn_01x03_Socket, J5 ICSP, SW1 SW_DIP_x02, U1 TPS613222ADBVR, U2 PIC16F13115-E/P

Commit message: Clean up bad footprints, make battery resistor divider DNP, and update PCB.
Parts:
- R7, R8: now not fitted
Changed lines of the file:
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@@
 		(on_board yes)
 		(in_pos_files yes)
-		(dnp no)
+		(dnp yes)
 		(fields_autoplaced yes)
 		(property "Reference" "R7"
@@
 		(on_board yes)
 		(in_pos_files yes)
-		(dnp no)
+		(dnp yes)
 		(fields_autoplaced yes)
 		(property "Reference" "R8"
