File: kicad/solar-light-charlie-boost/solar-light-charlie-boost.kicad_pcb (KiCad board)
At the start: 2 copper layers, 76.2 x 76.2 mm, 32 parts, among them J2 Conn_01x08_Socket, J3 Conn_01x03_Pin, J4 Conn_01x03_Socket, J5 ICSP, SW1 SW_DIP_x02, U1 TPS613221ADBVR, U2 PIC12F1572

Commit message: Clean up bad footprints, make battery resistor divider DNP, and update PCB.
Parts:
- added U1: TPS613222ADBVR, Package_TO_SOT_SMD:SOT-23-5_HandSoldering, F.Cu at (154.4, 117.7)
- U2: value PIC12F1572 -> PIC16F13115-E/P
- moved U2 0.22 mm to (123.9, 113.9)

Commit message: Move J5 to board front; relabel board
Parts:
- removed the U1 at (154.4, 117.7)
- J5: moved to F.Cu
- moved J5 12.7 mm to (132.2, 133.8)
Routing:
- net ICSPCLK: track 32.0 -> 33.0 mm
Other:
- board text added: "SOLAR DAISY Rev 2b"
- board text removed: "(c) 2026 Karen A Morrissey Carol J Wasinger SOLAR DAISY Rev 2a"
